File: eagle/tile-controller/tile-controller.sch (EAGLE design)
At the start: 24 parts, among them J1 AVR_SPI_PRG_6PTH

Commit message: Updated eagle version and added text labels R, W, B (red, white, black) for the weight input wire
Other:
- note added: "B"
- note added: "R"
- note added: "W"
Changed lines of the file:
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@@
 <?xml version="1.0" encoding="utf-8"?>
 <!DOCTYPE eagle SYSTEM "eagle.dtd">
-<eagle version="8.1.0">
+<eagle version="8.6.0">
 <drawing>
 <settings>
 <setting alwaysvectorfont="yes"/>
+<setting keepoldvectorfont="yes"/>
 <setting verticaltext="up"/>
 </settings>
@@
 <sheet>
 <plain>
+<text x="40.64" y="-25.4" size="1.778" layer="91">R</text>
+<text x="40.64" y="-27.94" size="1.778" layer="91">W</text>
+<text x="40.64" y="-30.48" size="1.778" layer="91">B</text>
 </plain>
 <instances>
